File: hardware/electronics/LogiBot PCB/LogiBot PCB.kicad_sch (KiCad schematic)
At the start: 55 parts, among them J1 XT60, J2 SWD Debug, J3 USB_C_Receptacle_USB2.0_16P, J4 UART Orange Pi, J5 Encoder, J6 BNO080 Module Conn, J7 J10_ESTOP, Q1 Q_PMOS_GSD, SW1 SW_Push, U1 LM2596S-5, U3 STM32G474RET6, U4 USBLC6-2SC6, U5 TJA1051T, U6 AP2112K-3.3, Y1 8MHz

Commit message: sc part2
Parts:
- removed C14, C16: 100nF, symbol Device:C
- removed C18: 4.7uF, symbol Device:C
- removed C6, C7: 22pF, symbol Device:C
- removed J2: SWD Debug, symbol Connector_Generic:Conn_01x04
- removed J4: UART Orange Pi, symbol Connector_Generic:Conn_01x04
- removed J5: Encoder, symbol Connector_Generic:Conn_01x06
- removed J6: BNO080 Module Conn, symbol Connector_Generic:Conn_01x08
- removed Y1: 8MHz, symbol Device:Crystal_GND24
- added C19, C20: 1uF, symbol Device:C
- added C21, C22: 22pF, symbol Device:C
- added D10: LED_STATUS L, symbol Device:LED
- added D9: LED_STATUS R, symbol Device:LED
- added J10: ENCODER_LEFT, symbol Connector_Generic:Conn_01x06
- added J11: ENCODER_RIGHT, symbol Connector_Generic:Conn_01x06
- added J12: J_IMU, symbol Connector_Generic:Conn_01x06
- added J13: VL53L0X, symbol Connector_Generic:Conn_01x06
- added J14: Ultrasonic Header, symbol Connector_Generic:Conn_01x04
- added J15: Bumper Switch, symbol Connector_Generic:Conn_01x02
- added J16: UART STM32 ↔ ORANGE PI, symbol Connector_Generic:Conn_01x04
- added J2: SWD Debug, symbol Connector_Generic:Conn_01x06
- added J8: MotorDriver_Left, symbol Connector_Generic:Conn_01x08
- added J9: MotorDriver_Right, symbol Connector_Generic:Conn_01x08
- added R10, R12, R16, R17: 4.7K, symbol Device:R
- added R11, R20, R21, R22, R23, R24: 10K, symbol Device:R
- added R13, R14, R15, R18, R19: 330, symbol Device:R
- added TP10: TP_ENC_R_A, symbol Connector:TestPoint
- added TP11: TP_ENC_R_B, symbol Connector:TestPoint
- added TP12: ENC_L_A, symbol Connector:TestPoint
- added TP13: ENC_R_A, symbol Connector:TestPoint
- added TP14: SDA, symbol Connector:TestPoint
- added TP15: IMU INT, symbol Connector:TestPoint
- added TP16: BUMPER, symbol Connector:TestPoint
- added TP17: ENC_L_B, symbol Connector:TestPoint
- added TP18: ENC_R_B, symbol Connector:TestPoint
- added TP19: SCL, symbol Connector:TestPoint
- added TP20: TP8 VL53_INT, symbol Connector:TestPoint
- added TP6: TP_PWM_L, symbol Connector:TestPoint
- added TP7: TP_PWM_R, symbol Connector:TestPoint
- added TP8: TP_ENC_L_A, symbol Connector:TestPoint
- added TP9: TP_ENC_L_B, symbol Connector:TestPoint
- added Y2: 8MHz, symbol Device:Crystal_GND24
- C11, C12, C3, C5: value 100nF -> 100pF
- R8: value 1K -> 330
- SW1: value SW_Push -> BUTTON_RST
Connections:
- net 24V_MOTOR is gone; now on net VDD: C10.2, C9.2, Q1.3 (D), TP1.1, U1.1 (VIN), U3.1 (VBAT)
- net VDDA is gone; now on net VDD: U3.29 (VDDA)
- net VSS is gone; now on net GND: U3.15 (VSS), U3.31 (VSS), U3.47 (VSS), U3.63 (VSS)
- net VSSA is gone; now on net GND: U3.27 (VSSA)
- net +5V: now also J8.3 (Pin_3), J9.3 (Pin_3)
- net 3V3: now also C11.2, C12.2, C3.2, C5.2, J12.1 (Pin_1), J13.6 (Pin_6), J16.1 (Pin_1), J2.4 (Pin_4), R20.2, R21.2, R22.2, R23.2, R24.1
- net 5V_MAIN: now also J10.1 (Pin_1), J11.1 (Pin_1), J14.1 (Pin_1)
- net GND: now also C1.2, C11.1, C12.1, C13.1, C15.2, C17.2, C2.2, C3.1, C5.1, D3.1 (K), D4.1 (K), D5.1 (K), D6.1 (K), R1.2, SW1.1, C19.2, C20.2, C21.1, C22.2, D10.1 (K), D9.1 (K), J10.2 (Pin_2), J11.2 (Pin_2), J12.2 (Pin_2), J13.5 (Pin_5), J14.2 (Pin_2), J15.2 (Pin_2), J16.4 (Pin_4), J2.5 (Pin_5), J8.2 (Pin_2), J9.2 (Pin_2), Y2.2 (G), Y2.4 (G); no longer D6.2 (A)
- net SWCLK: now also U3.36 (PB14), J2.2 (Pin_2)
- net SWDIO: now also U3.35 (PB13), J2.1 (Pin_1)
- net Shield: now also J10.6 (Pin_6), J11.6 (Pin_6)
- net VDD: now also C1.1, C13.2, C15.1, C17.1, C2.1, U3.28 (VREF+), C19.1, C20.1, R11.1
- net at R1.1: now also U3.61 (PB8-BOOT0)
- net PA0: now reaches U3.12 (PA0)
- net PA0: now also J8.8 (Pin_8), TP6.1
- net DIR_L: now reaches U3.13 (PA1)
- net DIR_L: now also J8.7 (Pin_7)
- net EN_L: now reaches U3.14 (PA2)
- net EN_L: now also J8.6 (Pin_6)
- net PA3: now reaches U3.17 (PA3)
- net PA3: now also J9.8 (Pin_8), TP7.1
- net DIR_R: now reaches U3.18 (PA4)
- net DIR_R: now also J9.7 (Pin_7)
- net EN_R: now reaches U3.19 (PA5)
- net EN_R: now also J9.6 (Pin_6)
- net PC13: now reaches U3.2 (PC13)
- net PC13: now also R13.1
- net PA6: now reaches U3.20 (PA6)
- net PA6: now also J13.2 (Pin_2)
- net PA7: now reaches U3.21 (PA7)
- net PA7: now also J13.1 (Pin_1), TP20.1
- net ENC_L_A: now reaches U3.24 (PB0)
- net ENC_L_A: now also J10.3 (Pin_3), R10.2, R20.1, TP12.1, TP8.1
- net ENC_L_B: now reaches U3.25 (PB1)
- net ENC_L_B: now also J10.4 (Pin_4), R12.2, R21.1, TP17.1, TP9.1
- net ENC_R_B: now reaches U3.26 (PB2)
- net ENC_R_B: now also J11.4 (Pin_4), R17.2, R23.1, TP11.1, TP18.1
- net I2C_IMU_SCL: now reaches U3.30 (PB10)
- net I2C_IMU_SCL: now also U3.59 (PB6), J12.4 (Pin_4), J13.3 (Pin_3), TP19.1
- net I2C_IMU_SDA: now reaches U3.33 (PB11)
- net I2C_IMU_SDA: now also U3.60 (PB7), J12.3 (Pin_3), J13.4 (Pin_4), TP14.1
- net PC9: now reaches U3.41 (PC9)
- net PC9: now also R18.2
- net PA8: now reaches U3.42 (PA8)
- net PA8: now also J12.6 (Pin_6)
- net INT: now reaches U3.43 (PA9)
- net INT: now also J12.5 (Pin_5), TP15.1
- net PA10: now reaches U3.44 (PA10)
- net PA10: now also J14.4 (Pin_4)
- net PA11: now reaches U3.45 (PA11)
- net PA11: now also J14.3 (Pin_3)
- net at U3.5 (PF0-OSC_IN): now also C21.2, Y2.1
- net PC10: now reaches U3.52 (PC10)
- net PC10: now also R19.2
- net PC11: now reaches U3.53 (PC11)
- net PC11: now also R15.1
- net PC12: now reaches U3.54 (PC12)
- net PC12: now also R14.1
- net ENC_R_A: now reaches U3.56 (PB3)
- net ENC_R_A: now also J11.3 (Pin_3), J2.6 (Pin_6), R16.2, R22.1, TP10.1, TP13.1
- net at U3.6 (PF1-OSC_OUT): now also C22.1, Y2.3
- net NRST: now reaches U3.7 (PG10-~{RST})
- net NRST: now also SW1.2, J2.3 (Pin_3), R11.2
- net at D3.2 (A): now also R13.2
- net at L1.2, U1.2 (OUT): now also D6.2 (A); no longer D6.1 (K)
- net at D5.2 (A): now also R15.2
- net at D4.2 (A): now also R14.2
- new net: D10.2 (A), R19.1
- new net: D9.2 (A), R18.1
- new net: J8.4 (Pin_4), R12.1
- new net: J8.5 (Pin_5), R10.1
- new net: J9.4 (Pin_4), R17.1
- new net: J9.5 (Pin_5), R16.1
- new net BUMPER: J15.1 (Pin_1), R24.2, TP16.1
- new net CURRENT_L: J8.1 (Pin_1)
- new net CURRENT_R: J9.1 (Pin_1)
- new net ENC_L_Z: J10.5 (Pin_5)
- new net ENC_R_Z: J11.5 (Pin_5)
- new net STM_RX: J16.2 (Pin_2)
- new net STM_TX: J16.3 (Pin_3)
Other:
- note added: "MCU CORE"
- note added: "MOTOR CONTROL"
- note added: "SENSOR SYSTEM"
- moved on the sheet: C1, C13, C15, C17, C2, D2, D3, D4, D5, D6, J3, R1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

Commit message: schematic v1 finish
Parts:
- removed J7: J10_ESTOP, symbol Connector_Generic:Conn_01x02
- removed R6, R7: 100K, symbol Device:R
- added C14, C6: 100nF, symbol Device:C
- added C7: 10uF, symbol Device:C
- added D11: LED_BLUE_UART, symbol Device:LED
- added D12: Safety LED, symbol Device:LED
- added D7: LED_GREEN_USB, symbol Device:LED
- added D8: LED_YELLOW_CAN, symbol Device:LED
- added FB1: FerriteBead, symbol Device:FerriteBead
- added J4: Konektor CAN, symbol Connector_Generic:Conn_01x04
- added J5: Emergency Stop Connector, symbol Connector_Generic:Conn_01x02
- added J6: Bumper Switch Connector, symbol Connector_Generic:Conn_01x03
- added J7: Safety Header, symbol Connector_Generic:Conn_01x04
- added JP2: Jumper_2_Open, symbol Jumper:Jumper_2_Open
- added R25, R26, R27, R28: 330, symbol Device:R
- added R29: 10k, symbol Device:R
- added SW2: E-Stop Switch, symbol Switch:SW_SPST
- added SW3: Bumper Switch, symbol Switch:SW_SPST
- added TP21: USB_DP, symbol Connector:TestPoint
- added TP22: USB_DM, symbol Connector:TestPoint
- added TP23: UART_TX, symbol Connector:TestPoint
- added TP24: UART_RX, symbol Connector:TestPoint
- added TP25: CANH, symbol Connector:TestPoint
- added TP26: CANL, symbol Connector:TestPoint
- R4: value 120R -> 120
- R5: value 10K -> 10k
Connections:
- net STM_RX is gone; now on net PC5: J16.2 (Pin_2)
- net STM_TX is gone; now on net PC4: J16.3 (Pin_3)
- net 3V3: now also R5.1, J6.1 (Pin_1), R25.2, R26.2, R27.2, R28.2, R29.2
- net 5V_MAIN: now also U5.3 (VCC), C6.2, J4.1 (Pin_1)
- net BUMPER: now also U3.39 (PC7), J6.2 (Pin_2), J7.3 (Pin_3), R29.1, SW3.2 (B)
- net GND: now also J3.A1 (GND), J3.A12 (GND), J3.B1 (GND), J3.B12 (GND), J3.S1 (SHIELD), R2.2, R3.2, U4.2 (GND), U5.2 (GND), U5.8 (S), C14.1, C6.1, C7.1, D12.1 (K), J4.2 (Pin_2), J5.2 (Pin_2), J6.3 (Pin_3), J7.4 (Pin_4), SW2.1 (A), SW3.1 (A)
- net PA11: now also U4.4 (I/O2), TP22.1; no longer J14.3 (Pin_3)
- net VDD: now also FB1.2; no longer C15.1, C19.1, C2.1, C20.1, U3.28 (VREF+), U3.29 (VDDA)
- net CAN1_TX: now reaches U5.1 (TXD)
- net CAN1_TX: now also U3.62 (PB9)
- net CAN1_RX: now reaches U5.4 (RXD)
- net CAN1_RX: now also U3.58 (PB5)
- net at U5.6 (CANL): now also R4.2, JP2.2 (B)
- net CANH: now reaches U5.7 (CANH)
- net CANH: now also R4.1, J4.4 (Pin_4), TP25.1
- net PC2: now reaches U3.10 (PC2)
- net PC2: now also D11.1 (K)
- net PC4: now reaches U3.22 (PC4)
- net PC4: now also TP23.1
- net PC5: now reaches U3.23 (PC5)
- net PC5: now also TP24.1
- net ESTOP: now reaches U3.38 (PC6)
- net ESTOP: now also R5.2, J5.1 (Pin_1), J7.2 (Pin_2), SW2.2 (B)
- net SAFETY_LED_GPIO: now reaches U3.40 (PC8)
- net SAFETY_LED_GPIO: now also D12.2 (A), R28.1
- net PA12: now reaches U3.46 (PA12)
- net PA12: now also U4.6 (I/O1), TP21.1
- net SAFETY_OUT: now reaches U3.51 (PA15)
- net SAFETY_OUT: now also J7.1 (Pin_1)
- net PC0: now reaches U3.8 (PC0)
- net PC0: now also D7.1 (K)
- net PC1: now reaches U3.9 (PC1)
- net PC1: now also D8.1 (K)
- net at R2.1: now also J3.B5 (CC2)
- net at U4.1 (I/O1): now also J3.A6 (D+), J3.B6 (D+)
- net at U4.3 (I/O2): now also J3.A7 (D-), J3.B7 (D-)
- net +5V USB: now reaches U4.5 (VBUS)
- net +5V USB: now also J3.A4 (VBUS), J3.A9 (VBUS), J3.B4 (VBUS), J3.B9 (VBUS), C14.2, C7.2
- net at R3.1: now also J3.A5 (CC1)
- new net: D7.2 (A), R25.1
- new net: D8.2 (A), R26.1
- new net: D11.2 (A), R27.1
- new net CANL: J4.3 (Pin_3), JP2.1 (A), TP26.1
- new net PA13: J14.3 (Pin_3)
- new net VDDA: C15.1, C19.1, C2.1, C20.1, FB1.1, U3.28 (VREF+), U3.29 (VDDA)
- no-connect marks 0 -> 11
Other:
- note added: "COMMUNICATION"
- note removed: "Battery Management"
- note removed: "Power"
- moved on the sheet: C1, C10, C11, C12, C13, C15, C17, C19, C2, C20, C21, C22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

Commit message: schematic jadi footprint belum finish
Parts:
- C1, C10, C11, C12, C13, C14, C15, C2, C21, C22, C3, C5, C6: footprint (none) -> Capacitor_SMD:C_0603_1608Metric
- C17, C19, C20, C4, C7, C8: footprint (none) -> Capacitor_SMD:C_0805_2012Metric
- C9: footprint (none) -> Capacitor_THT:CP_Radial_D10.0mm_P5.00mm
- D1: footprint (none) -> Diode_SMD:D_SMB
- D10, D11, D12, D2, D3, D4, D5, D7, D8, D9: footprint (none) -> LED_SMD:LED_0805_2012Metric
- D6: footprint (none) -> Diode_SMD:D_SMA
- FB1: footprint (none) -> Inductor_SMD:L_1206_3216Metric
- J1: footprint (none) -> Connector_AMASS:AMASS_XT60-M_1x02_P7.20mm_Vertical
- J10, J11, J12, J13: footprint (none) -> Connector_JST:JST_XH_B6B-XH-A_1x06_P2.50mm_Vertical
- J14, J16, J4, J7: footprint (none) -> Connector_JST:JST_XH_B4B-XH-A_1x04_P2.50mm_Vertical
- J15, J5: footprint (none) -> Connector_JST:JST_XH_B2B-XH-A_1x02_P2.50mm_Vertical
- J2: footprint (none) -> Connector_PinHeader_2.54mm:PinHeader_1x06_P2.54mm_Vertical
- J6: footprint (none) -> Connector_JST:JST_XH_B3B-XH-A_1x03_P2.50mm_Vertical
- J8, J9: footprint (none) -> Connector_JST:JST_XH_B8B-XH-A_1x08_P2.50mm_Vertical
- JP2: footprint (none) -> Jumper:SolderJumper-2_P1.3mm_Bridged2Bar_Pad1.0x1.5mm
- R1, R10, R11, R12, R13, R14, R15, R16, R17, R18, R19, R2, R20, R21, R22, R23, R24, R25, R26, R27, R28, R29, R3, R4, R5, R8, R9: footprint (none) -> Resistor_SMD:R_0603_1608Metric
- SW1: footprint (none) -> Button_Switch_THT:SW_PUSH_6mm
- SW2, SW3, TP1, TP10, TP11, TP12, TP13, TP14, TP15, TP16, TP17, TP18, TP19, TP2, TP20, TP21, TP22, TP23, TP24, TP25, TP26, TP3, TP4, TP5, TP6, TP7, TP8, TP9: footprint (none) -> TestPoint:TestPoint_Pad_D1.5mm
- Y2: footprint (none) -> Crystal:Crystal_SMD_3225-4Pin_3.2x2.5mm

Commit message: pcb v1 finished
Parts:
- added H1, H2, H3, H4: MountingHole, MountingHole:MountingHole_3.2mm_M3, symbol Mechanical:MountingHole
- F1: footprint (none) -> Fuse:Fuseholder_Blade_Mini_Keystone_3568
- J3: footprint (none) -> Connector_USB:USB_C_Receptacle_GCT_USB4105-xx-A_16P_TopMnt_Horizontal
- L1: footprint (none) -> INDP125125X600N:INDP125125X600N
- Q1: footprint (none) -> Package_TO_SOT_SMD:SOT-23
Connections:
- net +5V is gone; now on net 5V_MAIN: J8.3 (Pin_3), J9.3 (Pin_3)
- net 3V3 is gone; now on net VDD: C11.2, C12.2, C3.2, C4.2, C5.2, J12.1 (Pin_1), J13.6 (Pin_6), J16.1 (Pin_1), J2.4 (Pin_4), J6.1 (Pin_1), R20.2, R21.2, R22.2, R23.2, R24.1, R25.2, R26.2, R27.2, R28.2, R29.2, R5.1, R8.1, TP3.1, U6.5 (VOUT)
- net NRST: now also J2.2 (Pin_2); no longer J2.3 (Pin_3)
- net PA13: now also U3.49 (PA13)
- net SWCLK: now also J2.3 (Pin_3); no longer J2.2 (Pin_2)
- no-connect marks 11 -> 10
